File: hardware/elbsupply.kicad_pcb (KiCad board)
At the start: 2 copper layers, 105 x 64.4 mm, 86 parts, among them CON1 AVR-ISP-6, IC1 ATMEGA8-AI, M3 Screw_PAN_Head_M3, P1 OUT_POS, P2 OUT_GND, P3 POWER_IN, Q1 KST2907A, SW1 SW_L, SW2 SW_R, SW3 SW_OE, SW4 SW_MD, U1 LM393, U2 TPS54331DDA, U3 LT1490, U4 LM358, U5 TS78L05CS, U6 LT3083

Commit message: final reviision A routing done, need to add some logo
Routing:
- net GND: track 44.8 -> 56.8 mm, vias 26 -> 33
Other:
- board text added: "Left"
- board text added: "Limit"
- board text added: "Mode"
- board text added: "Output Enable"
- board text added: "Power"
- board text added: "Rev. A"
- board text added: "Right"
- board text added: "Set"
- board text added: "devthrash 2015"
- board text removed: "Current Limit"
